File: sparks/Gauge.kicad_pcb (KiCad board)
At the start: 2 copper layers, 85 x 85 mm, 31 parts, among them J1 USB, J2 Conn_01x05_Male, J3 STEPPER, J5 LEDS, SW1 S_MODE, U1 TSR12450, U2 Feather, U3 LM2917, U4 L293D

Commit message: Stuff
Parts:
- removed C1, C2: 20nF, Capacitor_THT:CP_Radial_Tantal_D4.5mm_P2.50mm
- removed C3: 1uF, Capacitor_THT:CP_Radial_Tantal_D4.5mm_P2.50mm
- removed R1, R4, R7: 10k, Resistor_THT:R_Axial_DIN0204_L3.6mm_D1.6mm_P7.62mm_Horizontal
- removed R2: 20k, Resistor_THT:R_Axial_DIN0204_L3.6mm_D1.6mm_P7.62mm_Horizontal
- removed R3: 100k, Potentiometer_THT:Potentiometer_Piher_PT-6-H_Horizontal
- removed R5: 470, Resistor_THT:R_Axial_DIN0204_L3.6mm_D1.6mm_P7.62mm_Horizontal
- removed R6: 4.7k, Resistor_THT:R_Axial_DIN0204_L3.6mm_D1.6mm_P7.62mm_Horizontal
- added 2k??1: R, Resistor_THT:R_Axial_DIN0204_L3.6mm_D1.6mm_P7.62mm_Horizontal, F.Cu at (160.0, 90.0)
- added 47k1: R, Resistor_THT:R_Axial_DIN0204_L3.6mm_D1.6mm_P7.62mm_Horizontal, F.Cu at (174.0, 79.6)
- D1: value D -> LED; footprint Diode_THT:D_DO-41_SOD81_P7.62mm_Horizontal -> LED_THT:LED_D5.0mm
- U3: value LM2917 -> 4N35; footprint Footprints:LM2917 -> Package_DIP:DIP-6_W7.62mm
- moved D1 17.4 mm to (174.0, 92.5)
- moved SW1 9.60 mm to (175.0, 105.5)
- moved U3 8.10 mm to (164.0, 79.6), turned to 90 degrees
- moved R8 7.26 mm to (180.1, 100.0)
- moved D4 3.23 mm to (141.0, 71.0), turned to 90 degrees
- moved D5 3.23 mm to (141.0, 67.0), turned to 90 degrees
- moved D6 2.00 mm to (141.0, 79.0)
- moved D7 2.00 mm to (141.0, 75.0)
- moved J5 2.00 mm to (125.0, 76.6)
- moved R10 2.00 mm to (129.0, 75.0)
- moved R11 2.00 mm to (129.0, 71.0)
- moved R12 2.00 mm to (129.0, 67.0)
- moved R9 2.00 mm to (129.0, 79.0)
Connections:
- D1 pad 1: GND -> Net-(D1-Pad1)
- J2 pad 3: Net-(J2-Pad3) -> Net-(D1-Pad1)
- U2 pad 0: Net-(U2-Pad0) -> (no net)
- U2 pad 1: Net-(U2-Pad1) -> (no net)
- U2 pad 14: Net-(U2-Pad14) -> (no net)
- U2 pad 15: Net-(R7-Pad1) -> Net-(47k1-Pad2)
- U2 pad 17: Net-(U2-Pad17) -> (no net)
- U2 pad 18: Net-(U2-Pad18) -> (no net)
- U2 pad 19: Net-(U2-Pad19) -> (no net)
- U2 pad 20: Net-(U2-Pad20) -> (no net)
- U2 pad 21: Net-(U2-Pad21) -> (no net)
- U2 pad 22: Net-(U2-Pad22) -> (no net)
- U2 pad 23: Net-(U2-Pad23) -> (no net)
- U2 pad 24: Net-(U2-Pad24) -> (no net)
- U2 pad 25: Net-(U2-Pad25) -> (no net)
- U2 pad 27: Net-(U2-Pad27) -> (no net)
- U2 pad 29: Net-(U2-Pad29) -> (no net)
- U2 pad 30: Net-(U2-Pad30) -> (no net)
- U3 pad 2: Net-(C2-Pad1) -> Net-(D1-Pad2)
- U3 pad 3: Net-(C3-Pad1) -> (no net)
- U3 pad 4: Net-(C3-Pad1) -> GND
- U3 pad 5: Net-(R7-Pad1) -> Net-(47k1-Pad2)
Routing:
- net Net-(47k1-Pad2): track 0.00 -> 112.0 mm
- net Net-(R7-Pad1): track 102.7 -> 0.00 mm
- net +12V: track 89.8 -> 59.8 mm
- net Net-(D1-Pad1): track 0.00 -> 28.6 mm
- net +3V3: track 135.1 -> 153.9 mm
- net Net-(C3-Pad1): track 18.0 -> 0.00 mm
- net Net-(SW1-Pad1): track 32.5 -> 22.5 mm
- net Net-(2k??1-Pad2): track 20.5 -> 11.9 mm
- net Net-(C2-Pad1): track 7.69 -> 0.00 mm
- net Net-(J2-Pad3): track 6.05 -> 0.00 mm
- net Net-(D5-Pad2): track 4.38 -> 8.58 mm
- net Net-(D4-Pad2): track 4.38 -> 8.58 mm
- net Net-(R5-Pad2): track 3.73 -> 0.00 mm
- net Net-(J2-Pad1): track 49.4 -> 47.6 mm
Other:
- outline, holes or cut-outs redrawn
- board text added: "12V"
- board text added: "5V"
- board text added: "AFR"
- board text added: "GND"
- board text added: "HIGH BEAM"
- board text added: "INDICATORS"
- board text added: "NEUTRAL"
- board text added: "OIL"
- board text added: "TACH"
