File: sparks/Gauge.sch (KiCad schematic (older format))
At the start: 31 parts, among them J1 USB, J2 Conn_01x05_Male, J3 STEPPER, J5 LEDS, SW1 S_MODE, U1 TSR12450, U2 Feather, U3 LM2917, U4 L293D

Commit message: Stuff
Parts:
- removed C1, C2: 20nF, Capacitor_THT:CP_Radial_Tantal_D4.5mm_P2.50mm, symbol Device:CP1_Small
- removed C3: 1uF, Capacitor_THT:CP_Radial_Tantal_D4.5mm_P2.50mm, symbol Device:CP1_Small
- removed D1: D, Diode_THT:D_DO-41_SOD81_P7.62mm_Horizontal, symbol Device:D_Small
- removed R1, R4, R7: 10k, Resistor_THT:R_Axial_DIN0204_L3.6mm_D1.6mm_P7.62mm_Horizontal, symbol Device:R_US
- removed R2: 20k, Resistor_THT:R_Axial_DIN0204_L3.6mm_D1.6mm_P7.62mm_Horizontal, symbol Device:R_US
- removed R3: 100k, Potentiometer_THT:Potentiometer_Piher_PT-6-H_Horizontal, symbol Device:R_Variable_US
- removed R5: 470, Resistor_THT:R_Axial_DIN0204_L3.6mm_D1.6mm_P7.62mm_Horizontal, symbol Device:R_US
- removed R6: 4.7k, Resistor_THT:R_Axial_DIN0204_L3.6mm_D1.6mm_P7.62mm_Horizontal, symbol Device:R_US
- removed U3: LM2917, Footprints:LM2917, symbol New_Library:LM2917
- added D?: D_Zener, symbol Device:D_Zener
- added R?: R, symbol Device:R
- U1: symbol New_Library:TSR12450 -> Gauge-rescue:TSR12450-New_Library
- U2: symbol New_Library:Feather -> Gauge-rescue:Feather-New_Library
- U4: symbol New_Library:L293D -> Gauge-rescue:L293D-New_Library
Connections:
- net GND: now also D?.2 (A)
- net at J2.3 (Pin_3): now also R?.1

Commit message: Stuff
Parts:
- removed D?: D_Zener, symbol Device:D_Zener
- added 47k: R, Resistor_THT:R_Axial_DIN0204_L3.6mm_D1.6mm_P7.62mm_Horizontal, symbol Device:R
- added D1: LED, LED_THT:LED_D5.0mm, symbol Device:LED
- added U3: 4N35, Package_DIP:DIP-6_W7.62mm, symbol Isolator:4N35
- 2k??1: renamed from R?; footprint (none) -> Resistor_THT:R_Axial_DIN0204_L3.6mm_D1.6mm_P7.62mm_Horizontal
Connections:
- net +12V: now also 2k??1.1
- net +3V3: now also 47k.1
- net GND: now also U3.4
- net at U2.15 (A1): now also 47k.2, U3.5
- net at J2.3 (Pin_3): now also D1.1 (K); no longer 2k??1.1
- net at 2k??1.2: now also U3.1
- new net: D1.2 (A), U3.2
Other:
- moved on the sheet: 2k??1
Changed lines of the file:
@@
 Connection ~ 6350 1300
 $Comp
-L Device:R R?
+L Device:R 2k??1
 U 1 1 5CC47B3E
-P 3450 2350
-F 0 "R?" V 3657 2350 50  0000 C CNN
-F 1 "R" V 3566 2350 50  0000 C CNN
-F 2 "" V 3380 2350 50  0001 C CNN
-F 3 "~" H 3450 2350 50  0001 C CNN
-	1    3450 2350
+P 3550 2050
+F 0 "2k??1" V 3757 2050 50  0000 C CNN
+F 1 "R" V 3666 2050 50  0000 C CNN
+F 2 "Resistor_THT:R_Axial_DIN0204_L3.6mm_D1.6mm_P7.62mm_Horizontal" V 3480 2050 50  0001 C CNN
+F 3 "~" H 3550 2050 50  0001 C CNN
+	1    3550 2050
 	0    -1   -1   0
-$EndComp
-$Comp
-L Device:D_Zener D?
-U 1 1 5CC47C89
-P 7850 2250
-F 0 "D?" V 7804 2329 50  0000 L CNN
-F 1 "D_Zener" V 7895 2329 50  0000 L CNN
-F 2 "" H 7850 2250 50  0001 C CNN
-F 3 "~" H 7850 2250 50  0001 C CNN
-	1    7850 2250
-	0    1    1    0
 $EndComp
 Wire Wire Line
 	1600 1700 1600 2350
-Wire Wire Line
-	4200 4550 2650 4550
 Wire Wire Line
 	1350 2450 1350 2350
@@
 	1600 2350 1600 3700
 Wire Wire Line
-	3150 1500 3150 2350
-Wire Wire Line
-	3150 2350 3300 2350
-Wire Wire Line
 	1600 1500 3150 1500
-Wire Wire Line
-	3600 2350 3700 2350
-Wire Wire Line
-	3700 2350 3700 2400
 $Comp
-L power:GND #PWR?
-U 1 1 5CC61241
-P 7850 2400
-F 0 "#PWR?" H 7850 2150 50  0001 C CNN
-F 1 "GND" H 7855 2227 50  0000 C CNN
-F 2 "" H 7850 2400 50  0001 C CNN
-F 3 "" H 7850 2400 50  0001 C CNN
-	1    7850 2400
+L Isolator:4N35 U3
+U 1 1 5CC6762B
+P 4000 2150
+F 0 "U3" H 4000 2475 50  0000 C CNN
+F 1 "4N35" H 4000 2384 50  0000 C CNN
+F 2 "Package_DIP:DIP-6_W7.62mm" H 3800 1950 50  0001 L CIN
+F 3 "https://www.vishay.com/docs/81181/4n35.pdf" H 4000 2150 50  0001 L CNN
+	1    4000 2150
 	1    0    0    -1
 $EndComp
+Wire Wire Line
+	3400 2050 2550 2050
+$Comp
+L Device:LED D1
+U 1 1 5CC6D33E
+P 3550 2450
+F 0 "D1" H 3541 2666 50  0000 C CNN
+F 1 "LED" H 3541 2575 50  0000 C CNN
+F 2 "LED_THT:LED_D5.0mm" H 3550 2450 50  0001 C CNN
+F 3 "~" H 3550 2450 50  0001 C CNN
+	1    3550 2450
+	1    0    0    -1
+$EndComp
+Wire Wire Line
+	3150 2450 3400 2450
+Wire Wire Line
+	3150 1500 3150 2450
+Wire Wire Line
+	3700 2450 3700 2250
+$Comp
+L power:GND #PWR0101
+U 1 1 5CC75146
+P 4300 2250
+F 0 "#PWR0101" H 4300 2000 50  0001 C CNN
+F 1 "GND" H 4305 2077 50  0000 C CNN
+F 2 "" H 4300 2250 50  0001 C CNN
+F 3 "" H 4300 2250 50  0001 C CNN
+	1    4300 2250
+	1    0    0    -1
+$EndComp
+Wire Wire Line
+	4300 2150 4750 2150
+Wire Wire Line
+	4750 2150 4750 4550
+Wire Wire Line
+	2650 4550 4750 4550
+$Comp
+L power:+3.3V #PWR0102
+U 1 1 5CC78434
+P 4750 1850
+F 0 "#PWR0102" H 4750 1700 50  0001 C CNN
+F 1 "+3.3V" H 4765 2023 50  0000 C CNN
+F 2 "" H 4750 1850 50  0001 C CNN
+F 3 "" H 4750 1850 50  0001 C CNN
+	1    4750 1850
+	1    0    0    -1
+$EndComp
+Connection ~ 4750 2150
+$Comp
+L Device:R 47k
+U 1 1 5CC782C8
+P 4750 2000
+F 0 "47k" H 4820 2046 50  0000 L CNN
+F 1 "R" H 4820 1955 50  0000 L CNN
+F 2 "Resistor_THT:R_Axial_DIN0204_L3.6mm_D1.6mm_P7.62mm_Horizontal" V 4680 2000 50  0001 C CNN
+F 3 "~" H 4750 2000 50  0001 C CNN
+	1    4750 2000
+	1    0    0    -1
+$EndComp
