File: circuit/circuit.kicad_pcb (KiCad board)
At the start: 2 copper layers, 85 x 85 mm, 25 parts, among them J1 USB, J2 Conn_01x05_Male, J3 STEPPER, J5 LEDS, SW1 S_MODE, U1 TSR12450, U2 Feather, U3 4N35, U4 L293D

Commit message: Stuff
Parts:
- U1: value TSR12450 -> TSR_1-2450; footprint Footprints:TSR1 -> Converter_DCDC:Converter_DCDC_TRACO_TSR-1_THT
- moved U1 2.63 mm to (137.0, 89.1)
Connections:
- U2 pad 2: GND -> (no net)
- U2 pad 26: +3V3 -> (no net)
- U2 pad 28: GND -> (no net)
- U2 pad 31: +5V -> (no net)
- U4 pad 5: GND -> (no net)
Routing:
- net +3V3: track 159.8 -> 154.3 mm
- net Net-(J1-Pad2): track 15.6 -> 14.5 mm
- net +5V: track 69.9 -> 68.8 mm
- removed copper zone on B.Cu, net GND
- removed copper zone on F.Cu, net GND
