File: circuit/circuit.sch (KiCad schematic (older format))
At the start: 23 parts, among them J1 USB, J2 Conn_01x05_Male, J3 STEPPER, J5 LEDS, SW1 S_MODE, U1 TSR12450, U2 Feather, U3 4N35, U4 L293D

Commit message: Stuff
Parts:
- removed R8: R_OIL_TEMP, Resistor_THT:R_Axial_DIN0204_L3.6mm_D1.6mm_P7.62mm_Horizontal, symbol Device:R_US
- added R1: R, Resistor_THT:R_Axial_DIN0204_L3.6mm_D1.6mm_P7.62mm_Horizontal, symbol Device:R
- added R3: 5.6k, Resistor_THT:R_Axial_DIN0204_L3.6mm_D1.6mm_P7.62mm_Horizontal, symbol Device:R
- added R4: 10k, Resistor_THT:R_Axial_DIN0204_L3.6mm_D1.6mm_P7.62mm_Horizontal, symbol Device:R
- R2: renamed from 47k; value R -> 47k
- R5: renamed from 2k??1; value R -> 2k
Connections:
- wire segments 94 -> 96
Changed lines of the file:
@@
 OIL TEMPERATURE
-$Comp
-L Device:R_US R8
-U 1 1 5CC082B2
-P 6350 1150
-F 0 "R8" H 6418 1196 50  0000 L CNN
-F 1 "R_OIL_TEMP" H 6418 1105 50  0000 L CNN
-F 2 "Resistor_THT:R_Axial_DIN0204_L3.6mm_D1.6mm_P7.62mm_Horizontal" V 6390 1140 50  0001 C CNN
-F 3 "~" H 6350 1150 50  0001 C CNN
-	1    6350 1150
-	1    0    0    -1
-$EndComp
 $Comp
 L Connector:Conn_01x04_Male J3
@@
 	3900 6300 6350 6300
 Wire Wire Line
-	6250 6400 6250 1400
-Wire Wire Line
-	6250 1400 1600 1400
-Wire Wire Line
-	3900 6400 6250 6400
+	3900 6400 5200 6400
 Wire Wire Line
 	6350 1300 1600 1300
 Wire Wire Line
 	6350 1300 6350 6300
-Connection ~ 6350 1300
-$Comp
-L Device:R 2k??1
+$Comp
+L Device:R R5
 U 1 1 5CC47B3E
 P 3550 2050
-F 0 "2k??1" V 3757 2050 50  0000 C CNN
-F 1 "R" V 3666 2050 50  0000 C CNN
+F 0 "R5" V 3757 2050 50  0000 C CNN
+F 1 "2k" V 3666 2050 50  0000 C CNN
 F 2 "Resistor_THT:R_Axial_DIN0204_L3.6mm_D1.6mm_P7.62mm_Horizontal" V 3480 2050 50  0001 C CNN
 F 3 "~" H 3550 2050 50  0001 C CNN
@@
 Connection ~ 4750 2150
 $Comp
-L Device:R 47k
+L Device:R R2
 U 1 1 5CC782C8
 P 4750 2000
-F 0 "47k" H 4820 2046 50  0000 L CNN
-F 1 "R" H 4820 1955 50  0000 L CNN
+F 0 "R2" H 4820 2046 50  0000 L CNN
+F 1 "47k" H 4820 1955 50  0000 L CNN
 F 2 "Resistor_THT:R_Axial_DIN0204_L3.6mm_D1.6mm_P7.62mm_Horizontal" V 4680 2000 50  0001 C CNN
 F 3 "~" H 4750 2000 50  0001 C CNN
@@
 	1    0    0    -1
 $EndComp
+$Comp
+L Device:R R3
+U 1 1 5CC4C352
+P 5700 3450
+F 0 "R3" H 5770 3496 50  0000 L CNN
+F 1 "5.6k" H 5770 3405 50  0000 L CNN
+F 2 "Resistor_THT:R_Axial_DIN0204_L3.6mm_D1.6mm_P7.62mm_Horizontal" V 5630 3450 50  0001 C CNN
+F 3 "~" H 5700 3450 50  0001 C CNN
+	1    5700 3450
+	1    0    0    -1
+$EndComp
+$Comp
+L Device:R R4
+U 1 1 5CC4C411
+P 5700 3750
+F 0 "R4" H 5770 3796 50  0000 L CNN
+F 1 "10k" H 5770 3705 50  0000 L CNN
+F 2 "Resistor_THT:R_Axial_DIN0204_L3.6mm_D1.6mm_P7.62mm_Horizontal" V 5630 3750 50  0001 C CNN
+F 3 "~" H 5700 3750 50  0001 C CNN
+	1    5700 3750
+	1    0    0    -1
+$EndComp
+Wire Wire Line
+	5700 3300 5700 1400
+Wire Wire Line
+	5700 1400 1600 1400
+$Comp
+L power:GND #PWR0103
+U 1 1 5CC4F079
+P 5700 3900
+F 0 "#PWR0103" H 5700 3650 50  0001 C CNN
+F 1 "GND" H 5705 3727 50  0000 C CNN
+F 2 "" H 5700 3900 50  0001 C CNN
+F 3 "" H 5700 3900 50  0001 C CNN
+	1    5700 3900
+	1    0    0    -1
+$EndComp
+Wire Wire Line
+	5700 3600 5200 3600
+Wire Wire Line
+	5200 3600 5200 6400
+Connection ~ 5700 3600
+$Comp
+L Device:R R1
+U 1 1 5CC5478B
+P 6350 1150
+F 0 "R1" H 6420 1196 50  0000 L CNN
+F 1 "R" H 6420 1105 50  0000 L CNN
+F 2 "Resistor_THT:R_Axial_DIN0204_L3.6mm_D1.6mm_P7.62mm_Horizontal" V 6280 1150 50  0001 C CNN
+F 3 "~" H 6350 1150 50  0001 C CNN
+	1    6350 1150
+	1    0    0    -1
+$EndComp
+Connection ~ 6350 1300
 $EndSCHEMATC

Commit message: Stuff
Parts:
- removed U1: TSR12450, Footprints:TSR1, symbol Gauge-rescue:TSR12450-New_Library
- removed U2: Feather, Footprints:Feather, symbol Gauge-rescue:Feather-New_Library
- removed U4: L293D, Footprints:L293D, symbol Gauge-rescue:L293D-New_Library
- added U?: TSR12450, symbol library:TSR12450
- added U?: L293D, symbol library:L293D
Connections:
- wire segments 96 -> 95
Changed lines of the file:
@@
 EESchema Schematic File Version 4
-LIBS:Gauge-cache
 EELAYER 26 0
 EELAYER END
@@
 $EndDescr
 $Comp
-L Gauge-rescue:L293D-New_Library U4
-U 1 1 5CB8E603
-P 8450 5050
-F 0 "U4" H 9028 5096 50  0000 L CNN
-F 1 "L293D" H 9028 5005 50  0000 L CNN
-F 2 "Footprints:L293D" H 8350 5050 50  0001 C CNN
-F 3 "" H 8350 5050 50  0001 C CNN
-	1    8450 5050
-	1    0    0    -1
-$EndComp
-$Comp
 L LED:CQY99 D4
 U 1 1 5CB8F18D
@@
 	1    0    0    -1
 $EndComp
-Wire Wire Line
-	8500 5650 8350 5650
-Connection ~ 8350 5650
 $Comp
 L power:GND #PWR0124
@@
 	8350 4350 7500 4350
 Connection ~ 8350 4350
-$Comp
-L Gauge-rescue:Feather-New_Library U2
-U 1 1 5CBFD77E
-P 3450 5850
-F 0 "U2" H 3450 6865 50  0000 C CNN
-F 1 "Feather" H 3450 6774 50  0000 C CNN
-F 2 "Footprints:Feather" H 3450 5850 50  0001 C CNN
-F 3 "" H 3450 5850 50  0001 C CNN
-	1    3450 5850
-	1    0    0    -1
-$EndComp
 Wire Wire Line
 	3900 5700 4100 5700
-$Comp
-L Gauge-rescue:TSR12450-New_Library U1
-U 1 1 5CC457F0
-P 2100 3450
-F 0 "U1" H 2100 3775 50  0000 C CNN
-F 1 "TSR12450" H 2100 3684 50  0000 C CNN
-F 2 "Footprints:TSR1" H 2100 3450 50  0001 C CNN
-F 3 "" H 2100 3450 50  0001 C CNN
-	1    2100 3450
-	1    0    0    -1
-$EndComp
 $Comp
 L Connector:Conn_01x04_Male J5
@@
 $EndComp
 Connection ~ 6350 1300
+$Comp
+L library:TSR12450 U?
+U 1 1 5CC85FA4
+P 2100 3450
+F 0 "U?" H 2100 3775 50  0000 C CNN
+F 1 "TSR12450" H 2100 3684 50  0000 C CNN
+F 2 "" H 2100 3450 50  0001 C CNN
+F 3 "" H 2100 3450 50  0001 C CNN
+	1    2100 3450
+	1    0    0    -1
+$EndComp
+$Comp
+L library:L293D U?
+U 1 1 5CC8619E
+P 8450 5050
+F 0 "U?" H 9028 5096 50  0000 L CNN
+F 1 "L293D" H 9028 5005 50  0000 L CNN
+F 2 "" H 8350 5050 50  0001 C CNN
+F 3 "" H 8350 5050 50  0001 C CNN
+	1    8450 5050
+	1    0    0    -1
+$EndComp
 $EndSCHEMATC

Commit message: Stuff
Parts:
- added U2: Feather, Footprints:Feather, symbol library:Feather
- U1: renamed from U?; footprint (none) -> Footprints:TSR1
- U4: renamed from U?; footprint (none) -> Footprints:L293D
Changed lines of the file:
@@
 EESchema Schematic File Version 4
+LIBS:circuit-cache
 EELAYER 26 0
 EELAYER END
@@
 Connection ~ 6350 1300
 $Comp
-L library:TSR12450 U?
+L library:TSR12450 U1
 U 1 1 5CC85FA4
 P 2100 3450
-F 0 "U?" H 2100 3775 50  0000 C CNN
+F 0 "U1" H 2100 3775 50  0000 C CNN
 F 1 "TSR12450" H 2100 3684 50  0000 C CNN
-F 2 "" H 2100 3450 50  0001 C CNN
+F 2 "Footprints:TSR1" H 2100 3450 50  0001 C CNN
 F 3 "" H 2100 3450 50  0001 C CNN
 	1    2100 3450
@@
 $EndComp
 $Comp
-L library:L293D U?
+L library:L293D U4
 U 1 1 5CC8619E
 P 8450 5050
-F 0 "U?" H 9028 5096 50  0000 L CNN
+F 0 "U4" H 9028 5096 50  0000 L CNN
 F 1 "L293D" H 9028 5005 50  0000 L CNN
-F 2 "" H 8350 5050 50  0001 C CNN
+F 2 "Footprints:L293D" H 8350 5050 50  0001 C CNN
 F 3 "" H 8350 5050 50  0001 C CNN
 	1    8450 5050
 	1    0    0    -1
 $EndComp
+$Comp
+L library:Feather U2
+U 1 1 5CCEA291
+P 3450 5850
+F 0 "U2" H 3450 6865 50  0000 C CNN
+F 1 "Feather" H 3450 6774 50  0000 C CNN
+F 2 "Footprints:Feather" H 3450 5850 50  0001 C CNN
+F 3 "" H 3450 5850 50  0001 C CNN
+	1    3450 5850
+	1    0    0    -1
+$EndComp

Commit message: Stuff
Parts:
- removed U1: TSR12450, Footprints:TSR1, symbol library:TSR12450
- added U1: TSR_1-2450, Converter_DCDC:Converter_DCDC_TRACO_TSR-1_THT, symbol Regulator_Switching:TSR_1-2450
Connections:
- net +12V: now also U1.1 (Vin)
- net GND: now also U1.2 (GND)
- net at J1.2 (Pin_2): now also U1.3 (Vout)
Changed lines of the file:
@@
 $EndComp
-Wire Wire Line
-	2100 3900 1600 3900
 Wire Wire Line
 	1600 3900 1600 3700
-Wire Wire Line
-	2450 3350 2450 4000
-Wire Wire Line
-	2450 4000 1400 4000
 Wire Wire Line
 	1400 4000 1400 3800
@@
 Connection ~ 1750 2050
 Wire Wire Line
-	1750 2050 1750 3350
+	1750 2050 1750 3250
 $Comp
 L Switch:SW_Push SW1
@@
 L power:+12V #PWR0114
 U 1 1 5CBD1F19
-P 2550 2050
-F 0 "#PWR0114" H 2550 1900 50  0001 C CNN
-F 1 "+12V" H 2565 2223 50  0000 C CNN
-F 2 "" H 2550 2050 50  0001 C CNN
-F 3 "" H 2550 2050 50  0001 C CNN
-	1    2550 2050
+P 3000 2050
+F 0 "#PWR0114" H 3000 1900 50  0001 C CNN
+F 1 "+12V" H 3015 2223 50  0000 C CNN
+F 2 "" H 3000 2050 50  0001 C CNN
+F 3 "" H 3000 2050 50  0001 C CNN
+	1    3000 2050
 	1    0    0    -1
 $EndComp
@@
 Wire Wire Line
 	2300 5400 2300 4250
-Wire Wire Line
-	2300 4250 2550 4250
-Wire Wire Line
-	2550 4250 2550 2050
-Connection ~ 2550 2050
-Wire Wire Line
-	1750 2050 2550 2050
 $Comp
 L Connector:Conn_01x05_Male J2
@@
 $EndComp
 Wire Wire Line
-	3400 2050 2550 2050
+	3400 2050 3000 2050
 $Comp
 L Device:LED D1
@@
 Connection ~ 6350 1300
 $Comp
-L library:TSR12450 U1
-U 1 1 5CC85FA4
-P 2100 3450
-F 0 "U1" H 2100 3775 50  0000 C CNN
-F 1 "TSR12450" H 2100 3684 50  0000 C CNN
-F 2 "Footprints:TSR1" H 2100 3450 50  0001 C CNN
-F 3 "" H 2100 3450 50  0001 C CNN
-	1    2100 3450
-	1    0    0    -1
-$EndComp
-$Comp
 L library:L293D U4
 U 1 1 5CC8619E
@@
 	1    0    0    -1
 $EndComp
+Wire Wire Line
+	3000 4250 3000 2050
+Wire Wire Line
+	2300 4250 3000 4250
+Connection ~ 3000 2050
+Wire Wire Line
+	1750 2050 3000 2050
+$Comp
+L Regulator_Switching:TSR_1-2450 U1
+U 1 1 5CD33323
+P 2350 3350
+F 0 "U1" H 2350 3717 50  0000 C CNN
+F 1 "TSR_1-2450" H 2350 3626 50  0000 C CNN
+F 2 "Converter_DCDC:Converter_DCDC_TRACO_TSR-1_THT" H 2350 3200 50  0001 L CIN
+F 3 "http://www.tracopower.com/products/tsr1.pdf" H 2350 3350 50  0001 C CNN
+	1    2350 3350
+	1    0    0    -1
+$EndComp
+Wire Wire Line
+	2750 4000 2750 3250
+Wire Wire Line
+	1400 4000 2750 4000
+Wire Wire Line
+	2350 3900 2350 3550
+Wire Wire Line
+	1600 3900 2350 3900
+Wire Wire Line
+	1950 3250 1750 3250
 $EndSCHEMATC
