File: v1/circuit/circuit.sch (KiCad schematic (older format))
At the start: 25 parts, among them J1 USB, J2 Conn_01x05_Male, J3 STEPPER, J5 LEDS, SW1 S_MODE, U1 TSR_1-2450, U2 Feather, U3 4N35, U4 L293D

Commit message: v1 and v2
Parts:
- U2: footprint Footprints:Feather -> footprints:Feather
Changed lines of the file:
@@
 F 0 "U2" H 3450 6865 50  0000 C CNN
 F 1 "Feather" H 3450 6774 50  0000 C CNN
-F 2 "Footprints:Feather" H 3450 5850 50  0001 C CNN
+F 2 "footprints:Feather" H 3450 5850 50  0001 C CNN
 F 3 "" H 3450 5850 50  0001 C CNN
 	1    3450 5850

Commit message: Stuff
Parts:
- removed J1: USB, Connector_PinHeader_2.54mm:PinHeader_1x02_P2.54mm_Vertical, symbol Connector:Conn_01x02_Male
- removed R10, R11, R12, R9: 220, Resistor_THT:R_Axial_DIN0204_L3.6mm_D1.6mm_P7.62mm_Horizontal, symbol Device:R
- removed U2: Feather, footprints:Feather, symbol library:Feather
- removed U4: L293D, Footprints:L293D, symbol library:L293D
- added U2: Feather, footprints:Feather, symbol symbol_library:Feather
- added U4: L293D, Package_DIP:DIP-16_W7.62mm, symbol Driver_Motor:L293D
- R1, R13, R14, R3, R4: footprint Resistor_THT:R_Axial_DIN0204_L3.6mm_D1.6mm_P7.62mm_Horizontal -> Resistor_THT:R_Axial_DIN0207_L6.3mm_D2.5mm_P10.16mm_Horizontal
- R2: value 47k -> 20k; footprint Resistor_THT:R_Axial_DIN0204_L3.6mm_D1.6mm_P7.62mm_Horizontal -> Resistor_THT:R_Axial_DIN0207_L6.3mm_D2.5mm_P10.16mm_Horizontal
- R5: value 2k -> 1k; footprint Resistor_THT:R_Axial_DIN0204_L3.6mm_D1.6mm_P7.62mm_Horizontal -> Resistor_THT:R_Axial_DIN0207_L6.3mm_D2.5mm_P10.16mm_Horizontal
Connections:
- net +3V3: now also U2.26 (3V3), U4.1 (EN1,2), U4.9 (EN3,4)
- net +5V: now also U1.3 (Vout), U2.31 (USB), U4.16 (VCC1), U4.8 (VCC2)
- net GND: now also U2.2 (GND), U2.28 (GND), U4.12 (GND), U4.13 (GND), U4.4 (GND), U4.5 (GND)
- net at D4.2 (A): now also J5.3 (Pin_3)
- net at D5.2 (A): now also J5.4 (Pin_4)
- net at D6.1 (K): now also J5.1 (Pin_1)
- net at D7.1 (K): now also J5.2 (Pin_2)
- net at SW1.1: now also U2.9
- net at R3.2, R4.1: now also U2.5
- net at J2.1 (Pin_1), R1.2: now also U2.6
- net at J3.1 (Pin_1): now also U4.14 (4Y)
- net at J3.2 (Pin_2): now also U4.11 (3Y)
- net at J3.3 (Pin_3): now also U4.6 (2Y)
- net at J3.4 (Pin_4): now also U4.3 (1Y)
- net at R2.2, U3.5: now also U2.15 (A1)
- net at R13.2, R14.1: now also U2.16 (A2)
- new net STEP_1: U2.13, U4.2 (1A)
- new net STEP_2: U2.12, U4.7 (2A)
- new net STEP_3: U2.11, U4.15 (4A)
- new net STEP_4: U2.10, U4.10 (3A)
Other:
- note removed: "5V"
- moved on the sheet: J3
