File: v2/circuit/circuit.kicad_pcb (KiCad board)
At the start: 2 copper layers, 90 x 90 mm, 36 parts, among them J1 Conn_01x05, J2 LEDS, M1 Stepper_Motor_bipolar, SW1 SW_Push, SW2 SW_Push, U1 ATmega328P-AU, U2 4N25, U3 HT1621B, U4 TSR_1-2450, U5 VIM-878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

Commit message: Stuff
Parts:
- removed D5, D6, D7: LED, LED_SMD:LED_0805_2012Metric
- removed LS1: Piezo, Fuse:Fuse_0201_0603Metric
- removed R10: 220, Resistor_SMD:R_0805_2012Metric
- removed RV1, RV3: R_POT, Potentiometer_THT:Potentiometer_Bourns_3266Y_Vertical
- removed SW1: SW_Push, Button_Switch_SMD:SW_SPST_B3S-1000
- added C4: C, Capacitor_THT:C_Disc_D3.0mm_W2.0mm_P2.50mm, F.Cu at (170.0, 95.0)
- added J3: Conn_01x01, footprints:wire-pad, F.Cu at (123.0, 85.0)
- added J4: Conn_01x01, footprints:wire-pad, F.Cu at (120.0, 85.0)
- added J5: Conn_01x01, footprints:wire-pad, F.Cu at (117.0, 85.0)
- added U7: FGPMMOPA6H, footprints:FGPMMOPA6H, F.Cu at (182.0, 101.7)
- J1: value Conn_01x05 -> Conn_01x01; footprint Connector_Molex:Molex_PicoBlade_53047-1010_1x05_P1.25mm_Vertical -> footprints:wire-pad; moved to F.Cu
- J2: value LEDS -> Conn_01x01; footprint Connector_PinHeader_2.54mm:PinHeader_1x04_P2.54mm_Vertical -> footprints:wire-pad; moved to F.Cu
- R7, R8, R9: value 220 -> R
- moved R6 62.3 mm to (139.0, 63.9), turned to 90 degrees
- moved R8 39.9 mm to (146.9, 73.0)
- moved R2 39.1 mm to (169.0, 105.1), turned to 270 degrees
- moved R9 31.1 mm to (150.9, 73.0), turned to 0 degrees
- moved J1 29.3 mm to (172.0, 90.0)
- moved J2 25.8 mm to (169.0, 90.0), turned to 0 degrees
- moved R7 24.3 mm to (179.0, 72.1), turned to 270 degrees
- moved C2 17.5 mm to (180.4, 87.9)
- moved C3 17.5 mm to (187.4, 87.9)
- moved Y1 17.5 mm to (181.4, 80.4)
- moved D4 11.0 mm to (170.0, 101.0)
- moved U1 5.49 mm to (169.8, 75.2)
- moved C1 5.10 mm to (167.0, 64.0), turned to 180 degrees
- moved R3 1.88 mm to (133.9, 77.0)
Connections:
- D4 pad 2: +5V -> Net-(D4-Pad2)
- J1 pad 1: GND -> /OIL_TEMP
- J2 pad 1: Net-(J2-Pad1) -> /AFR
- R2 pad 1: +5V -> Net-(D4-Pad1)
- R2 pad 2: Net-(R2-Pad2) -> GND
- R7 pad 1: Net-(J2-Pad1) -> +5V
- R7 pad 2: Net-(D4-Pad1) -> /OIL_TEMP
- R8 pad 1: Net-(J2-Pad2) -> +12V
- R8 pad 2: Net-(D5-Pad1) -> /BATTERY_VOLTAGE
- R9 pad 1: Net-(J2-Pad3) -> /BATTERY_VOLTAGE
- R9 pad 2: Net-(D6-Pad2) -> GND
- U1 pad 29: Net-(R2-Pad2) -> +5V
- U3 pad 1: /SEG7 -> /SEG8
- U3 pad 19: Net-(LS1-Pad2) -> (no net)
- U3 pad 2: /SEG6 -> /SEG9
- U3 pad 20: Net-(LS1-Pad1) -> (no net)
- U3 pad 3: /SEG5 -> /SEG10
- U3 pad 4: /SEG4 -> /SEG11
- U3 pad 41: /SEG15 -> /SEG7
- U3 pad 42: /SEG14 -> /SEG6
- U3 pad 43: /SEG13 -> /SEG5
- U3 pad 44: /SEG12 -> /SEG4
- U3 pad 45: /SEG11 -> /SEG3
- U3 pad 46: /SEG10 -> /SEG2
- U3 pad 47: /SEG9 -> /SEG1
- U3 pad 48: /SEG8 -> /SEG0
- U3 pad 5: /SEG3 -> /SEG12
- U3 pad 6: /SEG2 -> /SEG13
- U3 pad 7: /SEG1 -> /SEG14
- U3 pad 8: /SEG0 -> /SEG15
Routing:
- net Net-(M1-Pad3): track 0.00 -> 53.3 mm
- net Net-(M1-Pad4): track 0.00 -> 42.1 mm
- net Net-(RV2-Pad2): track 0.00 -> 40.1 mm, vias 0 -> 1
- net Net-(M1-Pad2): track 0.00 -> 28.6 mm
- net Net-(M1-Pad1): track 0.00 -> 28.6 mm
- net /COM2: track 0.00 -> 24.4 mm
- net /SEG15: track 0.00 -> 21.9 mm
- net /SEG0: track 0.00 -> 21.5 mm
- net /SEG1: track 0.00 -> 20.7 mm
- net /COM3: track 0.00 -> 20.7 mm
- net /SEG14: track 0.00 -> 20.2 mm
- net /SEG2: track 0.00 -> 19.9 mm
- net /SEG3: track 0.00 -> 19.1 mm
- net /SEG7: track 0.00 -> 18.9 mm
- net /COM1: track 0.00 -> 18.5 mm
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
Commit message: Stuff
Parts:
- added BT1: Battery_Cell, Battery:BatteryHolder_Keystone_3000_1x12mm, B.Cu at (180.0, 97.6)
- added C6: C, Capacitor_SMD:C_1206_3216Metric, F.Cu at (177.6, 108.8)
- added J6: Conn_02x03_Odd_Even, Connector_PinHeader_2.54mm:PinHeader_2x03_P2.54mm_Vertical, F.Cu at (132.0, 87.0)
- added R10: R, Resistor_SMD:R_1206_3216Metric, F.Cu at (179.6, 114.5)
- added R11: R, Resistor_SMD:R_1206_3216Metric, F.Cu at (160.0, 75.4)
- added U8: MIC5205-3.3YM5, Package_TO_SOT_SMD:SOT-23-5, F.Cu at (185.4, 111.5)
- C2, C3: value C_Small -> C; footprint Capacitor_THT:C_Disc_D3.0mm_W1.6mm_P2.50mm -> Capacitor_SMD:C_1206_3216Metric
- C4: footprint Capacitor_THT:C_Disc_D3.0mm_W2.0mm_P2.50mm -> Capacitor_SMD:C_1206_3216Metric
- D1, D2, D3, D4: footprint LED_SMD:LED_0805_2012Metric -> LED_SMD:LED_1206_3216Metric
- J1, J2, J3, J4, J5: moved to B.Cu
- R1, R2, R3, R4, R5, R6, R7, R8, R9: footprint Resistor_SMD:R_0805_2012Metric -> Resistor_SMD:R_1206_3216Metric
- moved R7 41.2 mm to (138.0, 68.4)
- moved J5 33.2 mm to (149.0, 76.0)
- moved J4 27.5 mm to (146.0, 76.0)
- moved J1 24.4 mm to (152.0, 76.0)
- moved J3 21.9 mm to (143.0, 76.0)
- moved J2 19.8 mm to (155.0, 76.0)
- moved D1 8.82 mm to (121.4, 85.0), turned to 180 degrees
- moved R3 8.65 mm to (133.0, 68.4), turned to 270 degrees
- moved D4 6.08 mm to (169.0, 95.0)
- moved C4 6.02 mm to (169.5, 89.0)
- moved C3 5.89 mm to (181.6, 86.9)
- moved R2 5.22 mm to (168.0, 99.9)
- moved D2 5.02 mm to (136.4, 120.9)
- moved D3 5.02 mm to (164.4, 120.9)
- moved R4 5.02 mm to (131.4, 120.9)
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Connections:
- C2 pad 1: GND -> /XTAL1
- C2 pad 2: /XTAL1 -> GND
- C3 pad 1: GND -> /XTAL2
- C3 pad 2: /XTAL2 -> GND
- U1 pad 14: /AFR -> (no net)
- U1 pad 17: (no net) -> /AFR
- U1 pad 19: (no net) -> Net-(J6-Pad3)
- U1 pad 27: (no net) -> /RX
- U1 pad 28: (no net) -> /TX
- U1 pad 29: +5V -> Net-(J6-Pad5)
- U6 pad 10: /STEP_3 -> /STEP_4
- U6 pad 15: /STEP_4 -> /STEP_2
- U6 pad 7: /STEP_2 -> /STEP_3
- U7 pad 10: (no net) -> /RX
- U7 pad 4: (no net) -> /VBACKUP
- U7 pad 9: (no net) -> /TX
Routing:
- net +5V: track 0.00 -> 231.9 mm, vias 0 -> 5
- net /STEP_3: track 0.00 -> 66.0 mm
- net /TACHO: track 0.00 -> 60.7 mm, vias 0 -> 2
- net /STEP_4: track 0.00 -> 60.2 mm
- net /OIL_TEMP: track 0.00 -> 60.1 mm, vias 0 -> 1
- net /STEP_1: track 0.00 -> 59.9 mm
- net /LCD_DATA: track 0.00 -> 58.2 mm, vias 0 -> 2
- net /LCD_CS: track 0.00 -> 56.5 mm, vias 0 -> 2
- net /LCD_RD: track 0.00 -> 56.5 mm, vias 0 -> 2
- net /LCD_WR: track 0.00 -> 56.4 mm, vias 0 -> 2
- net /STEP_2: track 0.00 -> 52.0 mm
- net Net-(J6-Pad5): track 0.00 -> 51.5 mm, vias 0 -> 2
- net Net-(J6-Pad3): track 0.00 -> 41.5 mm
- net /MODE_BUTTON: track 0.00 -> 38.3 mm
- net +12V: track 0.00 -> 33.0 mm, vias 0 -> 1
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- added copper zone on B.Cu, net GND
- added copper zone on F.Cu, net GND
Other:
- board size 90 x 90 mm -> 84 x 84 mm
- board text added: "12V"
- board text added: "AFR"
- board text added: "GND"
- board text added: "OIL TEMP"
- board text added: "TACHO"
