File: v2/circuit/circuit.sch (KiCad schematic (older format))
At the start: 36 parts, among them J1 Conn_01x05, J2 LEDS, M1 Stepper_Motor_bipolar, SW1 SW_Push, SW2 SW_Push, U1 ATmega328P-AU, U2 4N25, U3 HT1621B, U4 TSR_1-2450, U5 VIM-878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

Commit message: Stuff
Parts:
- removed D5, D6, D7: LED, LED_SMD:LED_0805_2012Metric, symbol Device:LED
- removed J1: Conn_01x05, Connector_Molex:Molex_PicoBlade_53047-1010_1x05_P1.25mm_Vertical, symbol Connector_Generic:Conn_01x05
- removed J2: LEDS, Connector_PinHeader_2.54mm:PinHeader_1x04_P2.54mm_Vertical, symbol Connector:Conn_01x04_Male
- removed LS1: Piezo, Fuse:Fuse_0201_0603Metric, symbol Device:Speaker_Crystal
- removed R10: 220, Resistor_SMD:R_0805_2012Metric, symbol Device:R
- removed RV1, RV3: R_POT, Potentiometer_THT:Potentiometer_Bourns_3266Y_Vertical, symbol Device:R_POT
- removed SW1: SW_Push, Button_Switch_SMD:SW_SPST_B3S-1000, symbol Switch:SW_Push
- added C4: C, Capacitor_THT:C_Disc_D3.0mm_W2.0mm_P2.50mm, symbol Device:C
- added J1, J2, J3, J4, J5: Conn_01x01, footprints:wire-pad, symbol Connector_Generic:Conn_01x01
- added U7: FGPMMOPA6H, footprints:FGPMMOPA6H, symbol symbol_library:FGPMMOPA6H
- R7, R8, R9: value 220 -> R
Connections:
- net +12V: now also R8.1, J4.1 (Pin_1)
- net +5V: now also R7.1, U1.29 (~RESET~/PC6); no longer D4.2 (A), R2.1
- net AFR: now also J2.1 (Pin_1)
- net BATTERY_VOLTAGE: now also R8.2, R9.1
- net GND: now also R2.2, R9.2, C4.2, J5.1 (Pin_1), U7.12 (GND), U7.19 (GND), U7.3 (GND), U7.8 (GND)
- net OIL_TEMP: now also R7.2, J1.1 (Pin_1)
- net SEG0: now also U3.48 (SEG8); no longer U3.8 (SEG0)
- net SEG1: now also U3.47 (SEG9); no longer U3.7 (SEG1)
- net SEG10: now also U3.3 (SEG5); no longer U3.46 (SEG10)
- net SEG11: now also U3.4 (SEG4); no longer U3.45 (SEG11)
- net SEG12: now also U3.5 (SEG3); no longer U3.44 (SEG12)
- net SEG13: now also U3.6 (SEG2); no longer U3.43 (SEG13)
- net SEG14: now also U3.7 (SEG1); no longer U3.42 (SEG14)
- net SEG15: now also U3.8 (SEG0); no longer U3.41 (SEG15)
- net SEG2: now also U3.46 (SEG10); no longer U3.6 (SEG2)
- net SEG3: now also U3.45 (SEG11); no longer U3.5 (SEG3)
- net SEG4: now also U3.44 (SEG12); no longer U3.4 (SEG4)
- net SEG5: now also U3.43 (SEG13); no longer U3.3 (SEG5)
- net SEG6: now also U3.42 (SEG14); no longer U3.2 (SEG6)
- net SEG7: now also U3.41 (SEG15); no longer U3.1 (SEG7)
- net SEG8: now also U3.1 (SEG7); no longer U3.48 (SEG8)
- net SEG9: now also U3.2 (SEG6); no longer U3.47 (SEG9)
- net at D4.1 (K): now also R2.1; no longer R7.2
- net at D1.1 (K): now also J3.1 (Pin_1)
- new net: D4.2 (A), U7.5 (3D-FIX)
- new net +3V3: C4.1, U7.1 (VCC)
Other:
- note removed: "HIGH BEAM"
- note removed: "INDICATORS"
- note removed: "NEUTRAL"
- note removed: "OIL PRESSURE"
- moved on the sheet: C2, C3, D2, D3, M1, R4, R5, R6, RV2, SW2, U3, U4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

Commit message: Stuff
Parts:
- removed C2, C3: C_Small, Capacitor_THT:C_Disc_D3.0mm_W1.6mm_P2.50mm, symbol Device:C_Small
- added BT1: Battery_Cell, Battery:BatteryHolder_Keystone_3000_1x12mm, symbol Device:Battery_Cell
- added C2, C3, C6: C, Capacitor_SMD:C_1206_3216Metric, symbol Device:C
- added J6: Conn_02x03_Odd_Even, Connector_PinHeader_2.54mm:PinHeader_2x03_P2.54mm_Vertical, symbol Connector_Generic:Conn_02x03_Odd_Even
- added R10, R11: R, Resistor_SMD:R_1206_3216Metric, symbol Device:R
- added U8: MIC5205-3.3YM5, Package_TO_SOT_SMD:SOT-23-5, symbol Regulator_Linear:MIC5205-3.3YM5
- C4: footprint Capacitor_THT:C_Disc_D3.0mm_W2.0mm_P2.50mm -> Capacitor_SMD:C_1206_3216Metric
- D1, D2, D3, D4: footprint LED_SMD:LED_0805_2012Metric -> LED_SMD:LED_1206_3216Metric
- R1, R2, R3, R4, R5, R6, R7, R8, R9: footprint Resistor_SMD:R_0805_2012Metric -> Resistor_SMD:R_1206_3216Metric
Connections:
- net +3V3: now also C6.2, U8.5 (OUT)
- net +5V: now also J6.2 (Pin_2), R10.1, R11.1, U8.1 (IN); no longer U1.29 (~RESET~/PC6)
- net AFR: now also U1.17 (PB5); no longer U1.14 (PB2)
- net GND: now also BT1.2 (-), C2.2, C3.2, C6.1, J6.6 (Pin_6), U8.2 (GND)
- net OIL_TEMP: now also J6.1 (Pin_1)
- net STEP_2: now also U6.15 (4A); no longer U6.7 (2A)
- net STEP_3: now also U6.7 (2A); no longer U6.10 (3A)
- net STEP_4: now also U6.10 (3A); no longer U6.15 (4A)
- net TACHO: now also J6.4 (Pin_4)
- net XTAL1: now also C2.1
- net XTAL2: now also C3.1
- net at U1.19 (ADC6): now also J6.3 (Pin_3)
- net RX: now reaches U1.27 (PC4)
- net RX: now also U7.10 (RX)
- net TX: now reaches U1.28 (PC5)
- net TX: now also U7.9 (TX)
- net VBACKUP: now reaches U7.4 (VBACKUP)
- net VBACKUP: now also BT1.1 (+)
- new net: J6.5 (Pin_5), R11.2, U1.29 (~RESET~/PC6)
- new net: R10.2, U8.3 (EN)
Other:
- note added: "does it need a ferrite?"
- note added: "is this different from MIC5225?"
- moved on the sheet: RV2, U3, U5
