File: v2/face/face.kicad_pcb (KiCad board)
At the start: 2 copper layers, 85 x 85 mm, 18 parts, among them J1 Conn_01x01, J2 Conn_01x01, J3 Conn_01x01, J4 Conn_01x01, J5 Conn_01x01, J6 Conn_01x01

Commit message: Stuff
Other:
- board size 85 x 85 mm -> 84 x 84 mm
- board text added: "12V"
- board text added: "GND"
- board text added: "HB"
- board text added: "N"
- board text added: "OP"
- board text added: "TS"
Changed lines of the file:
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@@
   (general
     (thickness 1.6)
-    (drawings 50)
+    (drawings 56)
     (tracks 52)
     (zones 0)
@@
       (drillshape 0)
       (scaleselection 1)
-      (outputdirectory "face_gerber"))
+      (outputdirectory "gerber"))
   )
   (net 0 "")
@@
       (xy 0.682068 -1.717439)) (layer F.SilkS) (width 0.01))
   )
-  (gr_line (start 174.5 114.5) (end 174.5 127.5) (layer Edge.Cuts) (width 0.15))
-  (gr_arc (start 127.5 114.5) (end 127.5 112.5) (angle -90) (layer Edge.Cuts) (width 0.15))
-  (gr_arc (start 127.5 127.5) (end 125.5 127.5) (angle -90) (layer Edge.Cuts) (width 0.15))
+  (gr_text OP (at 154 63.2 270) (layer B.SilkS)
+    (effects (font (size 1.5 1.5) (thickness 0.3)) (justify mirror))
+  )
+  (gr_text N (at 151 64 270) (layer B.SilkS)
+    (effects (font (size 1.5 1.5) (thickness 0.3)) (justify mirror))
+  )
+  (gr_text TS (at 148 63.2 270) (layer B.SilkS)
+    (effects (font (size 1.5 1.5) (thickness 0.3)) (justify mirror))
+  )
+  (gr_text HB (at 145 63.2 270) (layer B.SilkS)
+    (effects (font (size 1.5 1.5) (thickness 0.3)) (justify mirror))
+  )
+  (gr_text 12V (at 157 62.6 270) (layer B.SilkS)
+    (effects (font (size 1.5 1.5) (thickness 0.3)) (justify mirror))
+  )
+  (gr_text GND (at 142 62.4 270) (layer B.SilkS)
+    (effects (font (size 1.5 1.5) (thickness 0.3)) (justify mirror))
+  )
+  (gr_line (start 174 116.5) (end 174 125.5) (layer Edge.Cuts) (width 0.15))
+  (gr_arc (start 128 116.5) (end 128 114.5) (angle -90) (layer Edge.Cuts) (width 0.15))
+  (gr_arc (start 128 125.5) (end 126 125.5) (angle -90) (layer Edge.Cuts) (width 0.15))
   (gr_circle (center 150 139) (end 151.5 139) (layer Edge.Cuts) (width 0.15))
-  (gr_arc (start 172.5 127.5) (end 172.5 129.5) (angle -90) (layer Edge.Cuts) (width 0.15))
+  (gr_arc (start 172 125.5) (end 172 127.5) (angle -90) (layer Edge.Cuts) (width 0.15))
   (gr_circle (center 124 116) (end 124.45 116) (layer Edge.Cuts) (width 0.15))
-  (gr_line (start 125.5 114.5) (end 125.5 127.5) (layer Edge.Cuts) (width 0.15))
+  (gr_line (start 126 116.5) (end 126 125.5) (layer Edge.Cuts) (width 0.15))
   (gr_circle (center 183.77 80.5) (end 185.27 80.5) (layer Edge.Cuts) (width 0.15))
-  (gr_arc (start 172.5 114.5) (end 174.5 114.5) (angle -90) (layer Edge.Cuts) (width 0.15))
-  (gr_line (start 127.5 112.5) (end 172.5 112.5) (layer Edge.Cuts) (width 0.15))
+  (gr_arc (start 172 116.5) (end 174 116.5) (angle -90) (layer Edge.Cuts) (width 0.15))
+  (gr_line (start 128 114.5) (end 172 114.5) (layer Edge.Cuts) (width 0.15))
   (gr_circle (center 116.22 80.5) (end 117.72 80.5) (layer Edge.Cuts) (width 0.15))
   (gr_circle (center 150 100) (end 151 100) (layer Edge.Cuts) (width 0.15))
-  (gr_line (start 127.5 129.5) (end 172.5 129.5) (layer Edge.Cuts) (width 0.15))
+  (gr_line (start 128 127.5) (end 172 127.5) (layer Edge.Cuts) (width 0.15))
   (gr_line (start 110.53291 114.139821) (end 116.171066 112.0877) (layer F.SilkS) (width 0.5))
   (gr_line (start 108 99.774975) (end 114 99.774975) (layer F.SilkS) (width 0.5))
@@
     (effects (font (size 4 4) (thickness 0.3)))
   )
-  (gr_circle (center 150 100) (end 192.5 100) (layer Edge.Cuts) (width 0.15))
+  (gr_circle (center 150 100) (end 192 100) (layer Edge.Cuts) (width 0.15))
   (via (at 165 88) (size 0.8) (drill 0.4) (layers F.Cu B.Cu) (net 1))
   (segment (start 166.6 88) (end 165 88) (width 0.25) (layer F.Cu) (net 1) (status 10))
