File: circuit_mcu/circuit_mcu.kicad_pcb (KiCad board)
At the start: 2 copper layers, 86 x 86 mm, 32 parts, among them J1 Conn_01x06, J2 Conn_01x04, J3 Conn_01x04, J4 Conn_01x04, J6 Conn_02x03_Odd_Even, SW2 SW_Push, U1 ATmega328P-PU, U2 4N25, U4 TSR_1-2450, U7 L80-R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

Commit message: Removed unused LCD read net
Parts:
- J2: value Conn_01x04 -> Conn_01x03; footprint Connector_PinSocket_2.54mm:PinSocket_1x04_P2.54mm_Vertical -> Connector_PinSocket_2.54mm:PinSocket_1x03_P2.54mm_Vertical
Connections:
- J2 pad 2: /LCD_RD -> /LCD_WR
- J2 pad 3: /LCD_WR -> /LCD_DATA
- U1 pad 3: /LCD_RD -> (no net)
Routing:
- net /LCD_RD: track 13.3 -> 0.00 mm
- net /LCD_WR: track 13.3 -> 17.7 mm
- net /LCD_DATA: track 13.3 -> 12.2 mm
